File: ir_design/kicad/ir-ring.kicad_sch (KiCad schematic)
At the start: 27 parts, among them J1 PicoBlade/MX1.25 5p R/A THT, Q1 AO3400A, U1 SY7200A, U2 TEMT6200FX01

Commit message: feat(ir): J1 is C588276, JLCPCB now places every part
Genuine Molex 530480510 (5-pin PicoBlade R/A THT), 13 990 in stock. BOM
grows to 14 lines / 24 parts; nothing is left for hand assembly.

Co-Authored-By: Claude Opus 5.5 <noreply@anthropic.com>
Parts:
- J1: LCSC (none) -> C588276
Changed lines of the file:
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@@
 (text "LED STRING - 8 x JNJ 3535 850 nm, in series" (exclude_from_sim no) (at 43.18 147.32 0) (effects (font (size 1.524 1.524) (bold yes)) (justify left)))
 (text "TEST PADS - bring-up, back side" (exclude_from_sim no) (at 226.06 99.06 0) (effects (font (size 1.524 1.524) (bold yes)) (justify left)))
-(symbol (lib_id "Connector_Generic:Conn_01x05") (at 45.72 88.9 0) (mirror y) (unit 1) (exclude_from_sim no) (in_bom yes) (on_board yes) (dnp no)(property "Reference" "J1" (at 40.64 80.01 0) (effects (font (size 1.27 1.27))))(property "Value" "PicoBlade/MX1.25 5p R/A THT" (at 40.64 97.79 0) (effects (font (size 1.27 1.27))))(property "Footprint" "ir-ring:Molex_PicoBlade_53048-0510_1x05_P1.25mm_Horizontal_Ring0.275" (at 45.72 88.9 0) (effects (font (size 1.27 1.27)) (hide yes)))(property "Datasheet" "~" (at 45.72 88.9 0) (effects (font (size 1.27 1.27)) (hide yes)))(property "Description" "" (at 45.72 88.9 0) (effects (font (size 1.27 1.27)) (hide yes)))(property "LCSC" "" (at 45.72 88.9 0) (effects (font (size 1.27 1.27)) (hide yes)))(pin "1")(pin "2")(pin "3")(pin "4")(pin "5")(instances (project "ir-ring" (path "/cdf836e3-5e27-575e-8189-40b446b7a956" (reference "J1") (unit 1)))))
+(symbol (lib_id "Connector_Generic:Conn_01x05") (at 45.72 88.9 0) (mirror y) (unit 1) (exclude_from_sim no) (in_bom yes) (on_board yes) (dnp no)(property "Reference" "J1" (at 40.64 80.01 0) (effects (font (size 1.27 1.27))))(property "Value" "PicoBlade/MX1.25 5p R/A THT" (at 40.64 97.79 0) (effects (font (size 1.27 1.27))))(property "Footprint" "ir-ring:Molex_PicoBlade_53048-0510_1x05_P1.25mm_Horizontal_Ring0.275" (at 45.72 88.9 0) (effects (font (size 1.27 1.27)) (hide yes)))(property "Datasheet" "~" (at 45.72 88.9 0) (effects (font (size 1.27 1.27)) (hide yes)))(property "Description" "" (at 45.72 88.9 0) (effects (font (size 1.27 1.27)) (hide yes)))(property "LCSC" "C588276" (at 45.72 88.9 0) (effects (font (size 1.27 1.27)) (hide yes)))(pin "1")(pin "2")(pin "3")(pin "4")(pin "5")(instances (project "ir-ring" (path "/cdf836e3-5e27-575e-8189-40b446b7a956" (reference "J1") (unit 1)))))
 (symbol (lib_id "ir-ring:SY7200A") (at 152.4 88.9 0) (unit 1) (exclude_from_sim no) (in_bom yes) (on_board yes) (dnp no)(property "Reference" "U1" (at 152.4 80.01 0) (effects (font (size 1.27 1.27))))(property "Value" "SY7200A" (at 152.4 97.79 0) (effects (font (size 1.27 1.27))))(property "Footprint" "Package_TO_SOT_SMD:SOT-23-6" (at 152.4 88.9 0) (effects (font (size 1.27 1.27)) (hide yes)))(property "Datasheet" "~" (at 152.4 88.9 0) (effects (font (size 1.27 1.27)) (hide yes)))(property "Description" "" (at 152.4 88.9 0) (effects (font (size 1.27 1.27)) (hide yes)))(property "LCSC" "C107309" (at 152.4 88.9 0) (effects (font (size 1.27 1.27)) (hide yes)))(pin "6")(pin "4")(pin "2")(pin "1")(pin "5")(pin "3")(instances (project "ir-ring" (path "/cdf836e3-5e27-575e-8189-40b446b7a956" (reference "U1") (unit 1)))))
 (symbol (lib_id "Device:L") (at 175.26 76.2 0) (unit 1) (exclude_from_sim no) (in_bom yes) (on_board yes) (dnp no)(property "Reference" "L1" (at 177.79999999999998 74.93 0) (effects (font (size 1.27 1.27)) (justify left)))(property "Value" "33uH SWPA4030S330MT" (at 177.79999999999998 77.47 0) (effects (font (size 1.27 1.27)) (justify left)))(property "Footprint" "ir-ring:L_Sunlord_SWPA4030S" (at 175.26 76.2 0) (effects (font (size 1.27 1.27)) (hide yes)))(property "Datasheet" "~" (at 175.26 76.2 0) (effects (font (size 1.27 1.27)) (hide yes)))(property "Description" "" (at 175.26 76.2 0) (effects (font (size 1.27 1.27)) (hide yes)))(property "LCSC" "C83470" (at 175.26 76.2 0) (effects (font (size 1.27 1.27)) (hide yes)))(pin "1")(pin "2")(instances (project "ir-ring" (path "/cdf836e3-5e27-575e-8189-40b446b7a956" (reference "L1") (unit 1)))))

Commit message: feat(ir): D1 -> B5819W SL (C8598), a JLCPCB Basic part
Same SOD-123 footprint, 40 V 1 A, meets the design's >= 40 V rule over the
33 V open-LED clamp (headroom 27 V -> 7 V). Drops one Extended setup fee;
BOM is now 8 Basic / 6 Extended lines. L1 has no Basic equivalent (Basic
inductors are mA-rated multilayer parts), nor do U1, U2, D2-D9, J1.

Co-Authored-By: Claude Opus 5.5 <noreply@anthropic.com>
Parts:
- D1: value >=40V 1A -> B5819W 40V 1A; LCSC C77343 -> C8598
Changed lines of the file:
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@@
 (symbol (lib_id "ir-ring:SY7200A") (at 152.4 88.9 0) (unit 1) (exclude_from_sim no) (in_bom yes) (on_board yes) (dnp no)(property "Reference" "U1" (at 152.4 80.01 0) (effects (font (size 1.27 1.27))))(property "Value" "SY7200A" (at 152.4 97.79 0) (effects (font (size 1.27 1.27))))(property "Footprint" "Package_TO_SOT_SMD:SOT-23-6" (at 152.4 88.9 0) (effects (font (size 1.27 1.27)) (hide yes)))(property "Datasheet" "~" (at 152.4 88.9 0) (effects (font (size 1.27 1.27)) (hide yes)))(property "Description" "" (at 152.4 88.9 0) (effects (font (size 1.27 1.27)) (hide yes)))(property "LCSC" "C107309" (at 152.4 88.9 0) (effects (font (size 1.27 1.27)) (hide yes)))(pin "6")(pin "4")(pin "2")(pin "1")(pin "5")(pin "3")(instances (project "ir-ring" (path "/cdf836e3-5e27-575e-8189-40b446b7a956" (reference "U1") (unit 1)))))
 (symbol (lib_id "Device:L") (at 175.26 76.2 0) (unit 1) (exclude_from_sim no) (in_bom yes) (on_board yes) (dnp no)(property "Reference" "L1" (at 177.79999999999998 74.93 0) (effects (font (size 1.27 1.27)) (justify left)))(property "Value" "33uH SWPA4030S330MT" (at 177.79999999999998 77.47 0) (effects (font (size 1.27 1.27)) (justify left)))(property "Footprint" "ir-ring:L_Sunlord_SWPA4030S" (at 175.26 76.2 0) (effects (font (size 1.27 1.27)) (hide yes)))(property "Datasheet" "~" (at 175.26 76.2 0) (effects (font (size 1.27 1.27)) (hide yes)))(property "Description" "" (at 175.26 76.2 0) (effects (font (size 1.27 1.27)) (hide yes)))(property "LCSC" "C83470" (at 175.26 76.2 0) (effects (font (size 1.27 1.27)) (hide yes)))(pin "1")(pin "2")(instances (project "ir-ring" (path "/cdf836e3-5e27-575e-8189-40b446b7a956" (reference "L1") (unit 1)))))
-(symbol (lib_id "Device:D_Schottky") (at 185.42 85.09 180) (unit 1) (exclude_from_sim no) (in_bom yes) (on_board yes) (dnp no)(property "Reference" "D1" (at 185.42 81.28 0) (effects (font (size 1.27 1.27))))(property "Value" ">=40V 1A" (at 185.42 88.9 0) (effects (font (size 1.27 1.27))))(property "Footprint" "Diode_SMD:D_SOD-123" (at 185.42 85.09 0) (effects (font (size 1.27 1.27)) (hide yes)))(property "Datasheet" "~" (at 185.42 85.09 0) (effects (font (size 1.27 1.27)) (hide yes)))(property "Description" "" (at 185.42 85.09 0) (effects (font (size 1.27 1.27)) (hide yes)))(property "LCSC" "C77343" (at 185.42 85.09 0) (effects (font (size 1.27 1.27)) (hide yes)))(pin "1")(pin "2")(instances (project "ir-ring" (path "/cdf836e3-5e27-575e-8189-40b446b7a956" (reference "D1") (unit 1)))))
+(symbol (lib_id "Device:D_Schottky") (at 185.42 85.09 180) (unit 1) (exclude_from_sim no) (in_bom yes) (on_board yes) (dnp no)(property "Reference" "D1" (at 185.42 81.28 0) (effects (font (size 1.27 1.27))))(property "Value" "B5819W 40V 1A" (at 185.42 88.9 0) (effects (font (size 1.27 1.27))))(property "Footprint" "Diode_SMD:D_SOD-123" (at 185.42 85.09 0) (effects (font (size 1.27 1.27)) (hide yes)))(property "Datasheet" "~" (at 185.42 85.09 0) (effects (font (size 1.27 1.27)) (hide yes)))(property "Description" "" (at 185.42 85.09 0) (effects (font (size 1.27 1.27)) (hide yes)))(property "LCSC" "C8598" (at 185.42 85.09 0) (effects (font (size 1.27 1.27)) (hide yes)))(pin "1")(pin "2")(instances (project "ir-ring" (path "/cdf836e3-5e27-575e-8189-40b446b7a956" (reference "D1") (unit 1)))))
 (symbol (lib_id "Device:C") (at 111.76 76.2 0) (unit 1) (exclude_from_sim no) (in_bom yes) (on_board yes) (dnp no)(property "Reference" "C1" (at 114.30000000000001 74.93 0) (effects (font (size 1.27 1.27)) (justify left)))(property "Value" "10uF 25V" (at 114.30000000000001 77.47 0) (effects (font (size 1.27 1.27)) (justify left)))(property "Footprint" "Capacitor_SMD:C_0805_2012Metric" (at 111.76 76.2 0) (effects (font (size 1.27 1.27)) (hide yes)))(property "Datasheet" "~" (at 111.76 76.2 0) (effects (font (size 1.27 1.27)) (hide yes)))(property "Description" "" (at 111.76 76.2 0) (effects (font (size 1.27 1.27)) (hide yes)))(property "LCSC" "C15850" (at 111.76 76.2 0) (effects (font (size 1.27 1.27)) (hide yes)))(pin "1")(pin "2")(instances (project "ir-ring" (path "/cdf836e3-5e27-575e-8189-40b446b7a956" (reference "C1") (unit 1)))))
 (symbol (lib_id "Device:C") (at 127.0 76.2 0) (unit 1) (exclude_from_sim no) (in_bom yes) (on_board yes) (dnp no)(property "Reference" "C3" (at 129.54 74.93 0) (effects (font (size 1.27 1.27)) (justify left)))(property "Value" "100nF" (at 129.54 77.47 0) (effects (font (size 1.27 1.27)) (justify left)))(property "Footprint" "Capacitor_SMD:C_0805_2012Metric" (at 127.0 76.2 0) (effects (font (size 1.27 1.27)) (hide yes)))(property "Datasheet" "~" (at 127.0 76.2 0) (effects (font (size 1.27 1.27)) (hide yes)))(property "Description" "" (at 127.0 76.2 0) (effects (font (size 1.27 1.27)) (hide yes)))(property "LCSC" "C49678" (at 127.0 76.2 0) (effects (font (size 1.27 1.27)) (hide yes)))(pin "1")(pin "2")(instances (project "ir-ring" (path "/cdf836e3-5e27-575e-8189-40b446b7a956" (reference "C3") (unit 1)))))

Commit message: feat(ir): manufacturer, MPN and description on every placed part
The JLCPCB BOM now carries Quantity, Manufacturer, Manufacturer Part # and
Description after its four auto-mapped columns, so LCSC's BOM tool and other
distributors can match it too. The data lives in one MFR table in
07_schematic.py, keyed by LCSC number so it cannot disagree with PARTS, and
11_fab.py refuses to build a BOM with a placed part missing either field.

Co-Authored-By: Claude Opus 5.5 <noreply@anthropic.com>
Parts:
- C1: MPN (none) -> CL21A106KAYNNNE; Manufacturer (none) -> Samsung Electro-Mechanics
- C2: MPN (none) -> 1206B475K500NT; Manufacturer (none) -> FH
- C3: MPN (none) -> CC0805KRX7R9BB104; Manufacturer (none) -> YAGEO
- D1: MPN (none) -> B5819W SL; Manufacturer (none) -> JSCJ
- D2, D3, D4, D5, D6, D7, D8, D9: MPN (none) -> JNJ-L-3535EW120-85035D-SL-J2; Manufacturer (none) -> JNJOPTO
- J1: MPN (none) -> 530480510; Manufacturer (none) -> MOLEX
- L1: MPN (none) -> SWPA4030S330MT; Manufacturer (none) -> Sunlord
- Q1: MPN (none) -> AO3400A; Manufacturer (none) -> AOS
- R1a, R1b: MPN (none) -> WR08W4R02FTL; Manufacturer (none) -> Walsin
- R2: MPN (none) -> 0805W8F1004T5E; Manufacturer (none) -> UNI-ROYAL
- R3: MPN (none) -> 0805W8F1001T5E; Manufacturer (none) -> UNI-ROYAL
- R4, R6, R7: MPN (none) -> 0805W8F1003T5E; Manufacturer (none) -> UNI-ROYAL
- U1: MPN (none) -> SY7200AABC; Manufacturer (none) -> Silergy
- U2: MPN (none) -> TEMT6200FX01; Manufacturer (none) -> VISHAY
