File: ir_design/kicad/ir-ring.kicad_sch (KiCad schematic)
At the start: 27 parts, among them J1 PicoBlade/MX1.25 5p R/A THT, Q1 AO3400A, U1 SY7200A, U2 TEMT6200FX01

Commit message: feat(ir): flat-top 2835 emitter, C22447924, so JLCPCB machine-places it
JLCPCB charged hand-soldering and manual-assembly fees for the domed 3535
(C22447930), even on a top-side-only quote: its soft silicone dome cannot
take a pick-up nozzle. Every 3535 IR part JLCPCB stocks is domed, so the
emitter moves to JNJ-L-2835CW-85020D-S-Q2, a flat-top PLCC 2835.

It is better on three other counts. At ~0.93 mm it fits the stock 1.00 mm
lens clearance, so the lens array no longer has to be raised. It has two
unequal pads with the large one as the anode, so a backwards part is a
reversed diode instead of the short that burned R1a on the 3535. And it has
13.7k in stock against 1k. Rated 350 mA (100 mA is 29 %), 125 degrees, with
about the same radiant power per mA.

The new footprint follows the vendor land pattern, centred on the body, so the
emitters stay on the dome centres. Pin 1 matches the datasheet and JLCPCB's
library. There are three thermal vias in the anode pad: the fourth corner
would sit on the +5V back route under D2. The committed routes import onto
the new pads unchanged. DRC with schematic parity is clean, with no
dangling tracks. The anode-pad join in 09_place.py and the old 3535
footprint are gone.

Co-Authored-By: Claude Opus 5.5 <noreply@anthropic.com>
Parts:
- D2, D3, D4, D5, D6, D7, D8, D9: value IR 850nm 120deg -> IR 850nm 125deg; footprint ir-ring:LED_3535_JNJ_EW120 -> ir-ring:LED_2835_JNJ_CW; LCSC C22447930 -> C22447924; MPN JNJ-L-3535EW120-85035D-SL-J2 -> JNJ-L-2835CW-85020D-S-Q2
Other:
- note added: "LED STRING - 8 x JNJ 2835 850 nm, in series"
- note removed: "LED STRING - 8 x JNJ 3535 850 nm, in series"
